File: glowing-sunflower/glowing-sunflower.kicad_sch (KiCad schematic)
At the start: 0 parts

Commit message: add: schematic
Parts:
- added C1: 0.01uF, symbol Device:C_Small
- added C2: 470uF, symbol Device:C_Polarized_US
- added D1, D2, D3, D4, D5, D6, D7, D8: LED, symbol Device:LED
- added J1: Barrel_Jack, symbol Connector:Barrel_Jack
- added Q1: PN2222A, Package_TO_SOT_THT:TO-92_Inline, symbol Transistor_BJT:PN2222A
- added R1, R2, R3, R4, R5, R6, R7, R8: 100E, symbol Device:R_US
- added R9: 150E, symbol Device:R_US
- added U1: NE555P, Package_DIP:DIP-8_W7.62mm, symbol Timer:NE555P
Connections:
- new net: Q1.1 (E), R1.1, R2.1, R3.1, R4.1, R5.1, R6.1, R7.1, R8.1
- new net: D5.2 (A), R5.2
- new net: C1.2, C2.2, D1.1 (K), D2.1 (K), D3.1 (K), D4.1 (K), D5.1 (K), D6.1 (K), D7.1 (K), D8.1 (K), J1.2, U1.1 (GND)
- new net: D6.2 (A), R6.2
- new net: D7.2 (A), R7.2
- new net: D3.2 (A), R3.2
- new net: D4.2 (A), R4.2
- new net: C2.1, Q1.2 (B), R9.1, U1.2 (TR), U1.6 (THR)
- new net: R9.2, U1.3 (Q)
- new net: D8.2 (A), R8.2
- new net: D2.2 (A), R2.2
- new net: J1.1, Q1.3 (C), U1.4 (R), U1.8 (VCC)
- new net: C1.1, U1.5 (CV)
- new net: D1.2 (A), R1.2
- no-connect marks 0 -> 1
Other:
- company: (none) -> www.technomad.in
- title: (none) -> Glowing Sunflower

Commit message: update: fix C2 cap value
Parts:
- C2: value 470uF -> 1000uF
Changed lines of the file:
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@@
   )
   (symbol (lib_id "Device:C_Polarized_US") (at 110.49 92.71 0) (unit 1)
-    (in_bom yes) (on_board yes) (dnp no) (fields_autoplaced)
-    (property "Reference" "C2" (at 114.3 90.805 0)
+    (in_bom yes) (on_board yes) (dnp no)
+    (property "Reference" "C2" (at 114.3 93.98 0)
       (effects (font (size 1.27 1.27)) (justify left))
     )
-    (property "Value" "470uF" (at 114.3 93.345 0)
+    (property "Value" "1000uF" (at 111.76 96.52 0)
       (effects (font (size 1.27 1.27)) (justify left))
     )

Commit message: update: fix R9 resistor value
Parts:
- R9: value 150E -> 750E
Changed lines of the file:
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@@
   (title_block
     (title "Glowing Sunflower")
-    (date "2023-09-20")
-    (rev "1.0")
+    (date "2023-09-21")
+    (rev "1.2")
     (company "www.technomad.in")
   )
@@
       (effects (font (size 1.27 1.27)) (justify left))
     )
-    (property "Value" "150E" (at 152.4 64.77 0)
-      (effects (font (size 1.27 1.27)) (justify left))
-    )
+    (property "Value" "750E" (at 152.4 64.77 0)
+      (effects (font (size 1.27 1.27)) (justify left))
+    )
